File: schematics/schematics.sch (KiCad schematic (older format))
At the start: 7 parts

Commit message: schematic notes
Other:
- note added: "TODO: Doublecheck application notes for MAX489"
Changed lines of the file:
@@
 Wire Notes Line
 	7100 3350 7100 3250
+Text Notes 9650 950  2    50   ~ 0
+TODO: Doublecheck application notes for MAX489
+Text Notes 4850 900  2    50   ~ 0
+TODO: Doublecheck application notes for MAX489
 $EndSCHEMATC

Commit message: Schematic
Other:
- note added: "TODO: \nOPTIONAL\nKEYPAD"
- note added: "TODO:\nOPTIONAL\nCHAR DISP"
Changed lines of the file:
@@
 EESchema Schematic File Version 4
+LIBS:schematics-cache
 EELAYER 30 0
 EELAYER END
@@
 	5450 2150 4700 2150
 Wire Wire Line
-	7900 1950 6950 1950
-Wire Wire Line
-	7900 1950 8200 1650
-Wire Wire Line
-	8200 1650 8500 1650
-Wire Wire Line
-	6950 1650 8100 1650
-Wire Wire Line
-	8100 1650 8200 1750
-Wire Wire Line
-	8200 1750 8500 1750
+	7800 1950 6950 1950
+Wire Wire Line
+	7800 1950 8100 1650
+Wire Wire Line
+	8100 1650 8500 1650
+Wire Wire Line
+	6950 1650 8000 1650
+Wire Wire Line
+	8000 1650 8100 1750
+Wire Wire Line
+	8100 1750 8500 1750
 Wire Wire Line
 	8100 1850 8500 1850
@@
 Text Notes 4850 900  2    50   ~ 0
 TODO: Doublecheck application notes for MAX489
+Text Notes 2400 3100 0    50   ~ 0
+ TODO: \nOPTIONAL\nKEYPAD
+Text Notes 1550 3100 0    50   ~ 0
+TODO:\nOPTIONAL\nCHAR DISP
+Wire Notes Line
+	1500 2800 1500 3200
+Wire Notes Line
+	1500 3200 2000 3200
+Wire Notes Line
+	2000 3200 2000 2800
+Wire Notes Line
+	2000 2800 1500 2800
+Wire Notes Line
+	2350 2800 2350 3150
+Wire Notes Line
+	2350 3150 2800 3150
+Wire Notes Line
+	2800 3150 2800 2800
+Wire Notes Line
+	2350 2800 2800 2800
+Text Notes 10250 4650 0    50   ~ 0
+ TODO: \nOPTIONAL\nKEYPAD
+Text Notes 9400 4650 0    50   ~ 0
+TODO:\nOPTIONAL\nCHAR DISP
+Wire Notes Line
+	9350 4350 9350 4750
+Wire Notes Line
+	9350 4750 9850 4750
+Wire Notes Line
+	9850 4750 9850 4350
+Wire Notes Line
+	9850 4350 9350 4350
+Wire Notes Line
+	10200 4350 10200 4700
+Wire Notes Line
+	10200 4700 10650 4700
+Wire Notes Line
+	10650 4700 10650 4350
+Wire Notes Line
+	10200 4350 10650 4350
 $EndSCHEMATC

Commit message: all kinds of changes to random stuff
Other:
- note added: "TODO: ADD\nTERMINATION\nRESISTORS"
Changed lines of the file:
@@
 Wire Notes Line
 	10200 4350 10650 4350
+Text Notes 4500 1300 0    50   ~ 0
+TODO: ADD\nTERMINATION\nRESISTORS
+Text Notes 7550 1350 0    50   ~ 0
+TODO: ADD\nTERMINATION\nRESISTORS
 $EndSCHEMATC

Commit message: .
Parts:
- removed D?: D, symbol Device:D
- removed Q?: DMG2302U, Package_TO_SOT_SMD:SOT-23, symbol Transistor_FET:DMG2302U
- added D? (x16): DIODE, symbol pspice:DIODE
- added J?: RFID-RC522, symbol Connector:Conn_01x08_Male
- added J?: KEYPAD, symbol Connector:Conn_01x08_Male
- added LCD_2004A: Conn_01x16_Male, symbol Connector:Conn_01x16_Male
- added Q?: TIP120, Package_TO_SOT_THT:TO-220-3_Vertical, symbol Transistor_BJT:TIP120
- added R?: 10K, symbol Device:R
- added R? (x7): 330, symbol Device:R
- added R?: 1K, symbol Device:R
- added RV?: 10K, symbol Device:R_POT_TRIM_US
- added SW_0, SW_1, SW_2, SW_3, SW_4, SW_5, SW_6, SW_7, SW_8, SW_9, SW_A, SW_B, SW_C, SW_D, SW_P, SW_S: SW_SPST, symbol Switch:SW_SPST
- added U? (x2): L7805, symbol Regulator_Linear:L7805
Connections:
- net labels added: 3V3, 5V, BCM_14, BCM_15, BCM_18, GPIO_00, GPIO_02, GPIO_04, GPIO_13, GPIO_14, GPIO_15, GPIO_16, GPIO_17, GPIO_18, GPIO_19, GPIO_21, GPIO_22, GPIO_23, GPIO_25, GPIO_26, GPIO_27, GPIO_33, KP_C0, KP_C1, KP_C2, KP_C3, KP_R0, KP_R1, KP_R2, KP_R3
- net labels removed: PWM
- wire segments 64 -> 163
Other:
- note added: "3V3"
- note added: "ALL BCM IN INTERIOR\nGO TO RPI0W\n"
- note added: "ALL GPIO IN EXTERIOR\nGO TO NODEMCU\n"
- note added: "DB0"
- note added: "DB1\n"
- note added: "DB2"
- note added: "DB3"
- note added: "DB4"
- note added: "DB5"
- note added: "DB6"
- note added: "DB7"
- note added: "E"
- note added: "GND"
- note added: "IRQ"
- note added: "KP_C0"
- note added: "KP_C1"
- note added: "KP_C2"
- note added: "KP_C3"
- note added: "KP_R0"
- note added: "KP_R1"
- note added: "KP_R2"
- note added: "KP_R3"
- note added: "LED+"
- note added: "LED-"
- note added: "MAINS PSU\nRS-25-12"
- note added: "MISO"
- note added: "MOSI"
- note added: "Prevents crash on firmware upload\n no idea why…\n"
- note added: "RS"
- note added: "RST"
- note added: "RW"
- note added: "SCK"
- note added: "SDA"
- note added: "Someone should design a more \nefficient voltage converter here:"
- note added: "VCC"
- note added: "VD"
- note added: "VSS"
- note removed: "MAINS PSU"
- note removed: "TO PI0W"
- note removed: "TODO: COPY. \nARDUINO MINI"
- note removed: "TODO: COPY. \nMFRC522 REF"
- note removed: "TODO: COPY.\n 12v to 5v"
- note removed: "TODO: Doublecheck application notes for MAX489"
- note removed: "TODO: \nOPTIONAL\nKEYPAD"
- note removed: "TODO:\nDO WE NEED\nPROTECTION\nRESITORS HERE?"
- note removed: "TODO:\nOPTIONAL\nCHAR DISP"
- moved on the sheet: DOOR_LOCK_STRIKE, J?, U?

Commit message: .
Parts:
- added R? (x2): 330, symbol Device:R
- SW_0, SW_1, SW_2, SW_3, SW_4, SW_5, SW_6, SW_7, SW_8, SW_9, SW_A, SW_B, SW_C, SW_D, SW_P, SW_S: symbol Switch:SW_SPST -> Switch:SW_Push
- U? (x2): value L7805 -> VX7805
Connections:
- wire segments 163 -> 167
Other:
- note added: "ALL GPIO IN EXTERIOR\nGO TO NODEMCU\n / ESP32\n"
- note added: "Im not actually using diodes here\nbut if we had them we could\nprevent ghosting"
- note removed: "ALL GPIO IN EXTERIOR\nGO TO NODEMCU\n"
- note removed: "Someone should design a more \nefficient voltage converter here:"
- note removed: "TODO: ADD\nTERMINATION\nRESISTORS"
- moved on the sheet: DOOR_LOCK_STRIKE, U?

Commit message: .
Parts:
- removed R?: 330, symbol Device:R
- added Q?: PN2222A, Package_TO_SOT_THT:TO-92_Inline, symbol Transistor_BJT:PN2222A
- added R?: 1K, symbol Device:R
Connections:
- net labels added: GPIO_05
- wire segments 167 -> 168
Other:
- note added: "ALL GPIO IN EXTERIOR GO TO \nNODEMCU / ESP32. Will probably\nchange GPIO assignments in PCB"
- note added: "TODO: Could run DE to\nGPIO for future proofing"
- note removed: "ALL GPIO IN EXTERIOR\nGO TO NODEMCU\n / ESP32\n"
Changed lines of the file:
@@
 L power:GND #PWR?
 U 1 1 5FD28A2F
-P 2350 4250
-F 0 "#PWR?" H 2350 4000 50  0001 C CNN
-F 1 "GND" H 2355 4077 50  0000 C CNN
-F 2 "" H 2350 4250 50  0001 C CNN
-F 3 "" H 2350 4250 50  0001 C CNN
-	1    2350 4250
+P 2350 3500
+F 0 "#PWR?" H 2350 3250 50  0001 C CNN
+F 1 "GND" H 2355 3327 50  0000 C CNN
+F 2 "" H 2350 3500 50  0001 C CNN
+F 3 "" H 2350 3500 50  0001 C CNN
+	1    2350 3500
 	-1   0    0    1
 $EndComp
-Wire Wire Line
-	2350 4250 2350 5050
 Text Label 2250 4200 1    50   ~ 0
 5V
-$Comp
-L Device:R R?
-U 1 1 5FD45134
-P 2250 4400
-F 0 "R?" H 2320 4446 50  0001 L CNN
-F 1 "330" V 2250 4350 50  0000 L CNN
-F 2 "" V 2180 4400 50  0001 C CNN
-F 3 "~" H 2250 4400 50  0001 C CNN
-	1    2250 4400
-	1    0    0    -1
-$EndComp
-Wire Wire Line
-	2250 4250 2250 4200
-Wire Wire Line
-	2250 4550 2250 5050
 Wire Wire Line
 	3600 5050 3600 4550
@@
 BCM_15
 Text Notes 550  750  0    50   ~ 0
-ALL GPIO IN EXTERIOR\nGO TO NODEMCU\n / ESP32\n
+ALL GPIO IN EXTERIOR GO TO \nNODEMCU / ESP32.  Will probably\nchange GPIO assignments in PCB
 Text Notes 11000 700  2    50   ~ 0
 ALL BCM IN INTERIOR\nGO TO RPI0W\n
@@
 Text Notes 4850 6450 0    50   ~ 0
 Im not actually using diodes here\nbut if we had them we could\nprevent ghosting
+Wire Wire Line
+	2250 4200 2250 5050
+$Comp
+L Transistor_BJT:PN2222A Q?
+U 1 1 5FC50645
+P 2450 3700
+F 0 "Q?" H 2640 3746 50  0000 L CNN
+F 1 "PN2222A" H 2640 3655 50  0000 L CNN
+F 2 "Package_TO_SOT_THT:TO-92_Inline" H 2650 3625 50  0001 L CIN
+F 3 "http://www.fairchildsemi.com/ds/PN/PN2222A.pdf" H 2450 3700 50  0001 L CNN
+	1    2450 3700
+	-1   0    0    1
+$EndComp
+Wire Wire Line
+	2350 3900 2350 5050
+$Comp
+L Device:R R?
+U 1 1 5FC6BCFE
+P 2850 3700
+F 0 "R?" H 2920 3746 50  0001 L CNN
+F 1 "1K" V 2850 3650 50  0000 L CNN
+F 2 "" V 2780 3700 50  0001 C CNN
+F 3 "~" H 2850 3700 50  0001 C CNN
+	1    2850 3700
+	0    -1   -1   0
+$EndComp
+Wire Wire Line
+	2650 3700 2700 3700
+Text Label 3100 3700 0    50   ~ 0
+GPIO_05
+Wire Wire Line
+	3000 3700 3100 3700
+Text Notes 1200 1400 0    50   ~ 0
+TODO: Could run DE to\nGPIO for future proofing
 $EndSCHEMATC
